File: PCB/HA-V1.0/HA-V1.0.kicad_pcb (KiCad board)
At the start: 2 copper layers, 1 part, among them U1 ATMEGA328P-ANR

Commit message: Firmware- Scratch
Parts:
- added C1: 22pF, Capacitor_THT:C_Disc_D3.0mm_W1.6mm_P2.50mm, F.Cu at (135.0, 93.0)
- added C2: 22pF, Capacitor_THT:C_Disc_D3.0mm_W1.6mm_P2.50mm, F.Cu at (135.0, 98.0)
- added XT1: Crystal, Crystal:Crystal_HC52-U_Vertical, F.Cu at (140.0, 93.0)
Routing:
- net Net-(C2-Pad1): track 0.00 -> 18.1 mm
- net Net-(C1-Pad1): track 0.00 -> 17.6 mm
- net GND: track 0.00 -> 5.00 mm
Changed lines of the file:
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@@
     (thickness 1.6)
     (drawings 0)
-    (tracks 0)
+    (tracks 12)
     (zones 0)
-    (modules 1)
-    (nets 30)
+    (modules 4)
+    (nets 31)
   )
   (page A4)
@@
   (net 23 "Net-(U1-Pad10)")
   (net 24 "Net-(U1-Pad9)")
-  (net 25 "Net-(U1-Pad8)")
-  (net 26 "Net-(U1-Pad7)")
-  (net 27 "Net-(U1-Pad4)")
-  (net 28 "Net-(U1-Pad2)")
-  (net 29 "Net-(U1-Pad1)")
+  (net 25 "Net-(U1-Pad4)")
+  (net 26 "Net-(U1-Pad2)")
+  (net 27 "Net-(U1-Pad1)")
+  (net 28 GND)
+  (net 29 "Net-(C1-Pad1)")
+  (net 30 "Net-(C2-Pad1)")
   (net_class Default "This is the default net class."
     (clearance 0.2)
@@
     (uvia_dia 0.3)
     (uvia_drill 0.1)
+    (add_net GND)
+    (add_net "Net-(C1-Pad1)")
+    (add_net "Net-(C2-Pad1)")
     (add_net "Net-(U1-Pad1)")
     (add_net "Net-(U1-Pad10)")
@@
     (add_net "Net-(U1-Pad32)")
     (add_net "Net-(U1-Pad4)")
-    (add_net "Net-(U1-Pad7)")
-    (add_net "Net-(U1-Pad8)")
     (add_net "Net-(U1-Pad9)")
+  )
+  (module Crystal:Crystal_HC52-U_Vertical (layer F.Cu)
+    (at 140 93 270)
+    (descr "Crystal THT HC-52/U, http://www.kvg-gmbh.de/assets/uploads/files/product_pdfs/XS71xx.pdf")
+    (tags "THT crystal HC-52/U")
+    (fp_text reference XT1 (at 1.9 -2.85 90) (layer F.SilkS)
+      (effects (font (size 1 1) (thickness 0.15)))
+    )
+    (fp_text value Crystal (at 1.9 2.85 90) (layer F.Fab)
+      (effects (font (size 1 1) (thickness 0.15)))
+    )
+    (fp_arc (start 4.25 0) (end 4.25 -1.85) (angle 180) (layer F.SilkS) (width 0.12))
+    (fp_arc (start -0.45 0) (end -0.45 -1.85) (angle -180) (layer F.SilkS) (width 0.12))
+    (fp_arc (start 4.25 0) (end 4.25 -1.15) (angle 180) (layer F.Fab) (width 0.1))
+    (fp_arc (start -0.45 0) (end -0.45 -1.15) (angle -180) (layer F.Fab) (width 0.1))
+    (fp_arc (start 4.25 0) (end 4.25 -1.65) (angle 180) (layer F.Fab) (width 0.1))
+    (fp_arc (start -0.45 0) (end -0.45 -1.65) (angle -180) (layer F.Fab) (width 0.1))
+    (fp_line (start 6.4 -2.1) (end -2.6 -2.1) (layer F.CrtYd) (width 0.05))
+    (fp_line (start 6.4 2.1) (end 6.4 -2.1) (layer F.CrtYd) (width 0.05))
+    (fp_line (start -2.6 2.1) (end 6.4 2.1) (layer F.CrtYd) (width 0.05))
+    (fp_line (start -2.6 -2.1) (end -2.6 2.1) (layer F.CrtYd) (width 0.05))
+    (fp_line (start -0.45 1.85) (end 4.25 1.85) (layer F.SilkS) (width 0.12))
+    (fp_line (start -0.45 -1.85) (end 4.25 -1.85) (layer F.SilkS) (width 0.12))
+    (fp_line (start -0.45 1.15) (end 4.25 1.15) (layer F.Fab) (width 0.1))
+    (fp_line (start -0.45 -1.15) (end 4.25 -1.15) (layer F.Fab) (width 0.1))
+    (fp_line (start -0.45 1.65) (end 4.25 1.65) (layer F.Fab) (width 0.1))
+    (fp_line (start -0.45 -1.65) (end 4.25 -1.65) (layer F.Fab) (width 0.1))
+    (fp_text user %R (at 1.9 0 90) (layer F.Fab)
+      (effects (font (size 1 1) (thickness 0.15)))
+    )
+    (pad 2 thru_hole circle (at 3.8 0 270) (size 1.5 1.5) (drill 0.8) (layers *.Cu *.Mask)
+      (net 30 "Net-(C2-Pad1)"))
+    (pad 1 thru_hole circle (at 0 0 270) (size 1.5 1.5) (drill 0.8) (layers *.Cu *.Mask)
+      (net 29 "Net-(C1-Pad1)"))
+    (model ${KISYS3DMOD}/Crystal.3dshapes/Crystal_HC52-U_Vertical.wrl
+      (at (xyz 0 0 0))
+      (scale (xyz 1 1 1))
+      (rotate (xyz 0 0 0))
+    )
+  )
+  (module Capacitor_THT:C_Disc_D3.0mm_W1.6mm_P2.50mm (layer F.Cu)
+    (at 135 98 180)
+    (descr "C, Disc series, Radial, pin pitch=2.50mm, , diameter*width=3.0*1.6mm^2, Capacitor, http://www.vishay.com/docs/45233/krseries.pdf")
+    (tags "C Disc series Radial pin pitch 2.50mm  diameter 3.0mm width 1.6mm Capacitor")
+    (fp_text reference C2 (at 1.25 -2.05) (layer F.SilkS)
+      (effects (font (size 1 1) (thickness 0.15)))
+    )
+    (fp_text value 22pF (at 1.25 2.05) (layer F.Fab)
+      (effects (font (size 1 1) (thickness 0.15)))
+    )
+    (fp_text user %R (at 1.25 0) (layer F.Fab)
+      (effects (font (size 0.6 0.6) (thickness 0.09)))
+    )
+    (fp_line (start 3.55 -1.05) (end -1.05 -1.05) (layer F.CrtYd) (width 0.05))
+    (fp_line (start 3.55 1.05) (end 3.55 -1.05) (layer F.CrtYd) (width 0.05))
+    (fp_line (start -1.05 1.05) (end 3.55 1.05) (layer F.CrtYd) (width 0.05))
+    (fp_line (start -1.05 -1.05) (end -1.05 1.05) (layer F.CrtYd) (width 0.05))
+    (fp_line (start 0.621 0.92) (end 1.879 0.92) (layer F.SilkS) (width 0.12))
+    (fp_line (start 0.621 -0.92) (end 1.879 -0.92) (layer F.SilkS) (width 0.12))
+    (fp_line (start 2.75 -0.8) (end -0.25 -0.8) (layer F.Fab) (width 0.1))
+    (fp_line (start 2.75 0.8) (end 2.75 -0.8) (layer F.Fab) (width 0.1))
+    (fp_line (start -0.25 0.8) (end 2.75 0.8) (layer F.Fab) (width 0.1))
+    (fp_line (start -0.25 -0.8) (end -0.25 0.8) (layer F.Fab) (width 0.1))
+    (pad 2 thru_hole circle (at 2.5 0 180) (size 1.6 1.6) (drill 0.8) (layers *.Cu *.Mask)
+      (net 28 GND))
+    (pad 1 thru_hole circle (at 0 0 180) (size 1.6 1.6) (drill 0.8) (layers *.Cu *.Mask)
+      (net 30 "Net-(C2-Pad1)"))
+    (model ${KISYS3DMOD}/Capacitor_THT.3dshapes/C_Disc_D3.0mm_W1.6mm_P2.50mm.wrl
+      (at (xyz 0 0 0))
+      (scale (xyz 1 1 1))
+      (rotate (xyz 0 0 0))
+    )
+  )
+  (module Capacitor_THT:C_Disc_D3.0mm_W1.6mm_P2.50mm (layer F.Cu)
+    (at 135 93 180)
+    (descr "C, Disc series, Radial, pin pitch=2.50mm, , diameter*width=3.0*1.6mm^2, Capacitor, http://www.vishay.com/docs/45233/krseries.pdf")
+    (tags "C Disc series Radial pin pitch 2.50mm  diameter 3.0mm width 1.6mm Capacitor")
+    (fp_text reference C1 (at 1.25 -2.05) (layer F.SilkS)
+      (effects (font (size 1 1) (thickness 0.15)))
+    )
+    (fp_text value 22pF (at 1.25 2.05) (layer F.Fab)
+      (effects (font (size 1 1) (thickness 0.15)))
+    )
+    (fp_text user %R (at 1.25 0) (layer F.Fab)
+      (effects (font (size 0.6 0.6) (thickness 0.09)))
+    )
+    (fp_line (start 3.55 -1.05) (end -1.05 -1.05) (layer F.CrtYd) (width 0.05))
+    (fp_line (start 3.55 1.05) (end 3.55 -1.05) (layer F.CrtYd) (width 0.05))
+    (fp_line (start -1.05 1.05) (end 3.55 1.05) (layer F.CrtYd) (width 0.05))
+    (fp_line (start -1.05 -1.05) (end -1.05 1.05) (layer F.CrtYd) (width 0.05))
+    (fp_line (start 0.621 0.92) (end 1.879 0.92) (layer F.SilkS) (width 0.12))
+    (fp_line (start 0.621 -0.92) (end 1.879 -0.92) (layer F.SilkS) (width 0.12))
+    (fp_line (start 2.75 -0.8) (end -0.25 -0.8) (layer F.Fab) (width 0.1))
+    (fp_line (start 2.75 0.8) (end 2.75 -0.8) (layer F.Fab) (width 0.1))
+    (fp_line (start -0.25 0.8) (end 2.75 0.8) (layer F.Fab) (width 0.1))
+    (fp_line (start -0.25 -0.8) (end -0.25 0.8) (layer F.Fab) (width 0.1))
+    (pad 2 thru_hole circle (at 2.5 0 180) (size 1.6 1.6) (drill 0.8) (layers *.Cu *.Mask)
+      (net 28 GND))
+    (pad 1 thru_hole circle (at 0 0 180) (size 1.6 1.6) (drill 0.8) (layers *.Cu *.Mask)
+      (net 29 "Net-(C1-Pad1)"))
+    (model ${KISYS3DMOD}/Capacitor_THT.3dshapes/C_Disc_D3.0mm_W1.6mm_P2.50mm.wrl
+      (at (xyz 0 0 0))
+      (scale (xyz 1 1 1))
+      (rotate (xyz 0 0 0))
+    )
   )
   (module Package_QFP:QFP80P900X900X120-32N (layer F.Cu)
@@
       (net 24 "Net-(U1-Pad9)"))
     (pad 8 smd rect (at -4.3 2.8) (size 1.5 0.55) (layers F.Cu F.Paste F.Mask)
-      (net 25 "Net-(U1-Pad8)"))
+      (net 30 "Net-(C2-Pad1)"))
     (pad 7 smd rect (at -4.3 2) (size 1.5 0.55) (layers F.Cu F.Paste F.Mask)
-      (net 26 "Net-(U1-Pad7)"))
+      (net 29 "Net-(C1-Pad1)"))
     (pad 6 smd rect (at -4.3 1.2) (size 1.5 0.55) (layers F.Cu F.Paste F.Mask)
-      (net 27 "Net-(U1-Pad4)"))
+      (net 25 "Net-(U1-Pad4)"))
     (pad 5 smd rect (at -4.3 0.4) (size 1.5 0.55) (layers F.Cu F.Paste F.Mask)
       (net 12 "Net-(U1-Pad21)"))
     (pad 4 smd rect (at -4.3 -0.4) (size 1.5 0.55) (layers F.Cu F.Paste F.Mask)
-      (net 27 "Net-(U1-Pad4)"))
+      (net 25 "Net-(U1-Pad4)"))
     (pad 3 smd rect (at -4.3 -1.2) (size 1.5 0.55) (layers F.Cu F.Paste F.Mask)
       (net 12 "Net-(U1-Pad21)"))
     (pad 2 smd rect (at -4.3 -2) (size 1.5 0.55) (layers F.Cu F.Paste F.Mask)
-      (net 28 "Net-(U1-Pad2)"))
+      (net 26 "Net-(U1-Pad2)"))
     (pad 1 smd rect (at -4.3 -2.8) (size 1.5 0.55) (layers F.Cu F.Paste F.Mask)
-      (net 29 "Net-(U1-Pad1)"))
-  )
+      (net 27 "Net-(U1-Pad1)"))
+  )
+  (segment (start 132.5 93) (end 132.5 98) (width 0.25) (layer F.Cu) (net 28))
+  (segment (start 151.91 94.71) (end 144.71 94.71) (width 0.25) (layer F.Cu) (net 29))
+  (segment (start 144.71 94.71) (end 143 93) (width 0.25) (layer F.Cu) (net 29))
+  (segment (start 143 93) (end 140 93) (width 0.25) (layer F.Cu) (net 29))
+  (segment (start 140 93) (end 135 93) (width 0.25) (layer F.Cu) (net 29))
+  (segment (start 143 97) (end 140.2 97) (width 0.25) (layer F.Cu) (net 30))
+  (segment (start 151.91 95.51) (end 144.49 95.51) (width 0.25) (layer F.Cu) (net 30))
+  (segment (start 140.2 97) (end 140 96.8) (width 0.25) (layer F.Cu) (net 30))
+  (segment (start 144.49 95.51) (end 143 97) (width 0.25) (layer F.Cu) (net 30))
+  (segment (start 140 96.8) (end 138.2 96.8) (width 0.25) (layer F.Cu) (net 30))
+  (segment (start 137 98) (end 135 98) (width 0.25) (layer F.Cu) (net 30))
+  (segment (start 138.2 96.8) (end 137 98) (width 0.25) (layer F.Cu) (net 30))
 )

Commit message: Delete ATSD PROJ
Parts:
- added C5: 1000uF, Capacitor_THT:CP_Radial_D10.0mm_P5.00mm, F.Cu at (95.0, 105.0)
- added C6: 1000uF, Capacitor_THT:CP_Radial_D10.0mm_P5.00mm, F.Cu at (83.0, 106.0)
- added J1: Screw_Terminal_01x03, Connector_TE-Connectivity:TE_826576-3_1x03_P3.96mm_Vertical, F.Cu at (73.0, 96.0)
- added J3: Main_Relay, Connector_TE-Connectivity:TE_826576-2_1x02_P3.96mm_Vertical, F.Cu at (144.0, 78.0)
- added J4: Main_Relay, Connector_TE-Connectivity:TE_826576-2_1x02_P3.96mm_Vertical, F.Cu at (126.0, 115.4)
- U1: value ATMEGA328P-ANR -> ATmega328P-PU; footprint Package_QFP:QFP80P900X900X120-32N -> Package_DIP:DIP-28_W7.62mm
- moved U1 42.2 mm to (114.1, 89.6)
Connections:
- U1 pad 10: Net-(U1-Pad10) -> Net-(C1-Pad1)
- U1 pad 3: Net-(U1-Pad21) -> Net-(U1-Pad3)
- U1 pad 5: Net-(U1-Pad21) -> Net-(U1-Pad5)
- U1 pad 6: Net-(U1-Pad4) -> Net-(U1-Pad6)
- U1 pad 7: Net-(C1-Pad1) -> Net-(U1-Pad7)
- U1 pad 8: Net-(C2-Pad1) -> Net-(U1-Pad22)
- U1 pad 9: Net-(U1-Pad9) -> Net-(C2-Pad1)

Commit message: Final PCB Fabrication Done
Parts:
- removed C5, C6: 1000uF, Capacitor_THT:CP_Radial_D10.0mm_P5.00mm
- removed J3, J4: Main_Relay, Connector_TE-Connectivity:TE_826576-2_1x02_P3.96mm_Vertical
- added C3: 1000uF, Capacitor_THT:C_Radial_D10.0mm_H16.0mm_P5.00mm, F.Cu at (113.0, 105.5)
- added C4: 1000uF, Capacitor_THT:C_Radial_D10.0mm_H16.0mm_P5.00mm, F.Cu at (130.5, 91.5)
- added D1: 1N4007, Diode_THT:D_DO-41_SOD81_P10.16mm_Horizontal, F.Cu at (132.5, 112.5)
- added F1: Main, Fuse:Fuse_SunFuse-6HP, F.Cu at (66.5, 106.0)
- added J10: I2C_LCD, Connector_PinHeader_2.54mm:PinHeader_1x04_P2.54mm_Vertical, F.Cu at (139.0, 91.5)
- added J2: BUTTON, Connector_PinSocket_2.54mm:PinSocket_1x07_P2.54mm_Vertical, F.Cu at (171.5, 79.0)
- added PS1: AC_DC, Converter_ACDC:Converter_ACDC_MeanWell_IRM-10-xx_THT, F.Cu at (77.5, 84.5)
- added Q1: IRF540N, Package_TO_SOT_THT:TO-220-3_Vertical, F.Cu at (130.0, 105.5)
- added R1: 220, Resistor_THT:R_Axial_DIN0207_L6.3mm_D2.5mm_P7.62mm_Horizontal, F.Cu at (181.5, 113.5)
- added R10: 1K, Resistor_THT:R_Axial_DIN0207_L6.3mm_D2.5mm_P7.62mm_Horizontal, F.Cu at (164.5, 117.5)
- added R11: 1K, Resistor_THT:R_Axial_DIN0207_L6.3mm_D2.5mm_P7.62mm_Horizontal, F.Cu at (162.5, 103.5)
- added R2: 220, Resistor_THT:R_Axial_DIN0207_L6.3mm_D2.5mm_P7.62mm_Horizontal, F.Cu at (168.5, 117.5)
- added R3: 1K, Resistor_THT:R_Axial_DIN0207_L6.3mm_D2.5mm_P7.62mm_Horizontal, F.Cu at (185.0, 117.5)
- added R4: 1K, Resistor_THT:R_Axial_DIN0207_L6.3mm_D2.5mm_P7.62mm_Horizontal, F.Cu at (182.5, 101.5)
- added R5: 220, Resistor_THT:R_Axial_DIN0207_L6.3mm_D2.5mm_P7.62mm_Horizontal, F.Cu at (149.0, 119.5)
- added R6: 1K, Resistor_THT:R_Axial_DIN0207_L6.3mm_D2.5mm_P7.62mm_Horizontal, F.Cu at (152.5, 119.0)
- added R7: 1K, Resistor_THT:R_Axial_DIN0207_L6.3mm_D2.5mm_P7.62mm_Horizontal, F.Cu at (178.5, 97.5)
- added R8: 1K, Resistor_THT:R_Axial_DIN0207_L6.3mm_D2.5mm_P7.62mm_Horizontal, F.Cu at (142.5, 105.5)
- added RELAY: Main_Relay, Connector_TE-Connectivity:TE_826576-2_1x02_P3.96mm_Vertical, F.Cu at (125.5, 119.5)
- added RELAY_FB: Check Relay, Connector_TE-Connectivity:TE_826576-2_1x02_P3.96mm_Vertical, F.Cu at (139.0, 119.5)
- added SW1: U1_Reset, Button_Switch_THT:SW_PUSH_6mm_H4.3mm, F.Cu at (155.5, 95.0)
- added U2: PC817, Package_DIP:DIP-4_W7.62mm, F.Cu at (186.0, 113.5)
- added U3: PC817, Package_DIP:DIP-4_W7.62mm, F.Cu at (169.0, 113.5)
- added U4: PC817, Package_DIP:DIP-4_W7.62mm, F.Cu at (152.5, 112.0)
- added U5: L7805, Package_TO_SOT_THT:TO-220-3_Vertical, F.Cu at (125.0, 79.0)
- J1: value Screw_Terminal_01x03 -> MAINS; footprint Connector_TE-Connectivity:TE_826576-3_1x03_P3.96mm_Vertical -> Connector_Phoenix_MC_HighVoltage:PhoenixContact_MCV_1,5_2-G-5.08_1x02_P5.08mm_Vertical
- moved U1 38.7 mm to (151.5, 99.5), turned to 180 degrees
- moved C2 33.7 mm to (162.5, 78.5), turned to 0 degrees
- moved C1 33.1 mm to (162.5, 74.5), turned to 0 degrees
- moved XT1 26.2 mm to (158.5, 74.5)
- moved J1 18.8 mm to (55.5, 89.0), turned to 90 degrees
Connections:
- J1 pad 1: GND -> Net-(J1-Pad1)
- J1 pad 2: 5V-P -> Net-(F1-Pad2)
- U1 pad 1: Net-(U1-Pad1) -> 328P_RESET
- U1 pad 11: Net-(U1-Pad11) -> DOWN_BTN
- U1 pad 12: Net-(U1-Pad12) -> START_BTN
- U1 pad 16: Net-(U1-Pad16) -> RL_SIGNAL
- U1 pad 17: Net-(U1-Pad17) -> RC_SCN_U1
- U1 pad 20: Net-(U1-Pad20) -> 5V-P
- U1 pad 21: Net-(U1-Pad21) -> 5V-P
- U1 pad 22: Net-(U1-Pad22) -> GND
- U1 pad 27: Net-(U1-Pad27) -> LCD_SDA
- U1 pad 28: Net-(U1-Pad28) -> LCD_SCL
- U1 pad 4: Net-(U1-Pad4) -> SET_BTN
- U1 pad 5: Net-(U1-Pad5) -> OK_BTN
- U1 pad 6: Net-(U1-Pad6) -> UP_BTN
- U1 pad 7: Net-(U1-Pad7) -> 5V-P
- U1 pad 8: Net-(U1-Pad22) -> GND
Routing:
- net GND: track 5.00 -> 205.7 mm
- net 5V-P: track 0.00 -> 127.1 mm
- net RL_SIGNAL: track 0.00 -> 112.9 mm
- net 12V-P: track 0.00 -> 65.6 mm
- net RC_SCN_U1: track 0.00 -> 58.3 mm
- net Net-(Q1-Pad1): track 0.00 -> 40.7 mm
- net DOWN_BTN: track 0.00 -> 32.3 mm
- net START_BTN: track 0.00 -> 30.4 mm
- net Net-(R2-Pad2): track 0.00 -> 24.1 mm
- net Net-(J1-Pad1): track 0.00 -> 23.9 mm
- net Net-(F1-Pad2): track 0.00 -> 23.3 mm
- net Net-(R2-Pad1): track 0.00 -> 23.3 mm
- net Net-(F1-Pad1): track 0.00 -> 20.3 mm
- net OK_BTN: track 0.00 -> 20.1 mm
- net UP_BTN: track 0.00 -> 20.1 mm
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Other:
- board outline added: 158.5 x 69 mm
- board text added: "Controller"
- board text added: "HA V1.0"
- board text added: "L"
- board text added: "N"
- board text added: "S. ROY."
